File: _autosave-Projet_s6_oscillovpresquefinal.kicad_sch (KiCad schematic)
At the start: 34 parts, among them IC1 PGA849RGTR, J1 Conn_Coaxial, J2 Conn_01x06_Socket, J3 PILES_3AA, J4 Conn_01x05_Pin, SW1 SW_SPST, U1 MCP6001-OT, U2 AP2112K-3.3, U3 MCP1640x-xCHY, U4 STM32L476RGTx

Commit message: Résolution de toutes les erreurs ERC
Connections:
- net V_out_ecr is gone; now on net V3.3_DIG: C8.1, C8.2, D1.2 (K), U4.19 (VDD)
- net GND: no longer IC1.10 (REF), U1.1, U1.4 (-)
- new net Vref_1.5: IC1.10 (REF), U1.1, U1.4 (-)
Changed lines of the file:
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@@
 	)
 	(junction
+		(at 44.45 45.72)
+		(diameter 0)
+		(color 0 0 0 0)
+	)
+	(junction
 		(at 240.03 233.68)
 		(diameter 0)
@@
 	)
 	(junction
-		(at 226.06 243.84)
+		(at 208.28 196.85)
 		(diameter 0)
 		(color 0 0 0 0)
 	)
 	(junction
-		(at 292.1 229.87)
+		(at 226.06 243.84)
 		(diameter 0)
 		(color 0 0 0 0)
 	)
 	(junction
-		(at 151.13 68.58)
+		(at 292.1 229.87)
 		(diameter 0)
 		(color 0 0 0 0)
@@
 	(wire
 		(pts
+			(xy 44.45 45.72) (xy 46.99 45.72)
+		)
+		(stroke
+			(width 0)
+			(type default)
+		)
+	)
+	(wire
+		(pts
 			(xy 74.93 53.34) (xy 83.82 53.34)
 		)
@@
 	(wire
 		(pts
+			(xy 208.28 196.85) (xy 208.28 201.93)
+		)
+		(stroke
+			(width 0)
+			(type default)
+		)
+	)
+	(wire
+		(pts
 			(xy 226.06 247.65) (xy 241.3 247.65)
 		)
@@
 	(wire
 		(pts
+			(xy 44.45 43.18) (xy 44.45 45.72)
+		)
+		(stroke
+			(width 0)
+			(type default)
+		)
+	)
+	(wire
+		(pts
 			(xy 292.1 229.87) (xy 292.1 233.68)
 		)
@@
 	(wire
 		(pts
+			(xy 212.09 196.85) (xy 208.28 196.85)
+		)
+		(stroke
+			(width 0)
+			(type default)
+		)
+	)
+	(wire
+		(pts
 			(xy 240.03 228.6) (xy 269.24 228.6)
 		)
@@
 	(wire
 		(pts
-			(xy 151.13 68.58) (xy 151.13 72.39)
+			(xy 354.33 63.5) (xy 356.87 63.5)
 		)
 		(stroke
@@
 	(wire
 		(pts
-			(xy 354.33 63.5) (xy 356.87 63.5)
+			(xy 41.91 45.72) (xy 44.45 45.72)
 		)
 		(stroke
@@
 	(wire
 		(pts
-			(xy 228.6 208.28) (xy 236.22 208.28)
+			(xy 229.87 208.28) (xy 236.22 208.28)
 		)
 		(stroke
@@
 	(wire
 		(pts
+			(xy 208.28 196.85) (xy 207.01 196.85)
+		)
+		(stroke
+			(width 0)
+			(type default)
+		)
+	)
+	(wire
+		(pts
 			(xy 215.9 251.46) (xy 215.9 248.92)
 		)
@@
 		)
 	)
-	(global_label "V_out_ecr"
+	(global_label "V3.3_DIG"
 		(shape input)
 		(at 68.58 227.33 0)
@@
 		)
 		(property "Intersheetrefs" "${INTERSHEET_REFS}"
-			(at 80.5761 227.33 0)
+			(at 79.79 227.33 0)
 			(effects
 				(font
@@
 	(global_label "switch_Out"
 		(shape output)
-		(at 207.01 196.85 0)
+		(at 212.09 196.85 0)
 		(fields_autoplaced yes)
 		(effects
@@
 		)
 		(property "Intersheetrefs" "${INTERSHEET_REFS}"
-			(at 220.0947 196.85 0)
+			(at 225.1747 196.85 0)
 			(effects
 				(font
@@
 		)
 	)
-	(global_label "V_out_ecr"
+	(global_label "V3.3_DIG"
 		(shape input)
 		(at 341.63 62.23 90)
@@
 		)
 		(property "Intersheetrefs" "${INTERSHEET_REFS}"
-			(at 341.63 50.2339 90)
+			(at 341.63 51.02 90)
 			(effects
 				(font
@@
 	)
 	(symbol
+		(lib_id "power:PWR_FLAG")
+		(at 208.28 201.93 180)
+		(unit 1)
+		(exclude_from_sim no)
+		(in_bom yes)
+		(on_board yes)
+		(dnp no)
+		(fields_autoplaced yes)
+		(property "Reference" "#FLG02"
+			(at 208.28 203.835 0)
+			(effects
+				(font
+					(size 1.27 1.27)
+				)
+				(hide yes)
+			)
+		)
+		(property "Value" "PWR_FLAG"
+			(at 208.28 207.01 0)
+			(effects
+				(font
+					(size 1.27 1.27)
+				)
+			)
+		)
+		(property "Footprint" ""
+			(at 208.28 201.93 0)
+			(effects
+				(font
+					(size 1.27 1.27)
+				)
+				(hide yes)
+			)
+		)
+		(property "Datasheet" "~"
+			(at 208.28 201.93 0)
+			(effects
+				(font
+					(size 1.27 1.27)
+				)
+				(hide yes)
+			)
+		)
+		(property "Description" "Special symbol for telling ERC where power comes from"
+			(at 208.28 201.93 0)
+			(effects
+				(font
+					(size 1.27 1.27)
+				)
+				(hide yes)
+			)
+		)
+		(pin "1"
+		)
+		(instances
+			(project ""
+				(path "/79a95597-2db4-4373-9cc6-70296586f172"
+					(reference "#FLG02")
+					(unit 1)
+				)
+			)
+		)
+	)
+	(symbol
 		(lib_id "Device:C_Small")
 		(at 359.41 67.31 0)
@@
 	(symbol
 		(lib_id "power:GND")
-		(at 228.6 208.28 270)
+		(at 229.87 208.28 270)
 		(unit 1)
 		(exclude_from_sim no)
@@
 		(fields_autoplaced yes)
 		(property "Reference" "#PWR013"
-			(at 222.25 208.28 0)
+			(at 223.52 208.28 0)
 			(effects
 				(font
@@
 		)
 		(property "Value" "GND"
-			(at 224.79 208.2799 90)
+			(at 226.06 208.2799 90)
 			(effects
 				(font
@@
 		)
 		(property "Footprint" ""
-			(at 228.6 208.28 0)
+			(at 229.87 208.28 0)
 			(effects
 				(font
@@
 		)
 		(property "Datasheet" ""
-			(at 228.6 208.28 0)
+			(at 229.87 208.28 0)
 			(effects
 				(font
@@
 		)
 		(property "Description" "Power symbol creates a global label with name \"GND\" , ground"
-			(at 228.6 208.28 0)
+			(at 229.87 208.28 0)
 			(effects
 				(font
@@
 	(symbol
 		(lib_id "power:GND")
-		(at 46.99 45.72 270)
+		(at 41.91 45.72 270)
 		(unit 1)
 		(exclude_from_sim no)
@@
 		(fields_autoplaced yes)
 		(property "Reference" "#PWR01"
-			(at 40.64 45.72 0)
+			(at 35.56 45.72 0)
 			(effects
 				(font
@@
 		)
 		(property "Value" "GND"
-			(at 43.18 45.7199 90)
+			(at 38.1 45.7199 90)
 			(effects
 				(font
@@
 		)
 		(property "Footprint" ""
-			(at 46.99 45.72 0)
+			(at 41.91 45.72 0)
 			(effects
 				(font
@@
 		)
 		(property "Datasheet" ""
-			(at 46.99 45.72 0)
+			(at 41.91 45.72 0)
 			(effects
 				(font
@@
 		)
 		(property "Description" "Power symbol creates a global label with name \"GND\" , ground"
-			(at 46.99 45.72 0)
+			(at 41.91 45.72 0)
 			(effects
 				(font
@@
 	(symbol
 		(lib_id "power:GND")
-		(at 151.13 72.39 0)
-		(unit 1)
-		(exclude_from_sim no)
-		(in_bom yes)
-		(on_board yes)
-		(dnp no)
-		(fields_autoplaced yes)
-		(property "Reference" "#PWR06"
-			(at 151.13 78.74 0)
-			(effects
-				(font
-					(size 1.27 1.27)
-				)
-				(hide yes)
-			)
-		)
-		(property "Value" "GND"
-			(at 151.13 77.47 0)
-			(effects
-				(font
-					(size 1.27 1.27)
-				)
-			)
-		)
-		(property "Footprint" ""
-			(at 151.13 72.39 0)
-			(effects
-				(font
-					(size 1.27 1.27)
-				)
-				(hide yes)
-			)
-		)
-		(property "Datasheet" ""
-			(at 151.13 72.39 0)
-			(effects
-				(font
-					(size 1.27 1.27)
-				)
-				(hide yes)
-			)
-		)
-		(property "Description" "Power symbol creates a global label with name \"GND\" , ground"
-			(at 151.13 72.39 0)
-			(effects
-				(font
-					(size 1.27 1.27)
-				)
-				(hide yes)
-			)
-		)
-		(pin "1"
-		)
-		(instances
-			(project ""
-				(path "/79a95597-2db4-4373-9cc6-70296586f172"
-					(reference "#PWR06")
-					(unit 1)
-				)
-			)
-		)
-	)
-	(symbol
-		(lib_id "power:GND")
 		(at 180.34 219.71 0)
 		(unit 1)
@@
 					(unit 1)
 				)
+			)
+		)
+	)
+	(symbol
+		(lib_id "power:PWR_FLAG")
+		(at 44.45 43.18 0)
+		(unit 1)
+		(exclude_from_sim no)
+		(in_bom yes)
+		(on_board yes)
+		(dnp no)
+		(fields_autoplaced yes)
+		(property "Reference" "#FLG03"
+			(at 44.45 41.275 0)
+			(effects
+				(font
+					(size 1.27 1.27)
+				)
+				(hide yes)
+			)
+		)
+		(property "Value" "PWR_FLAG"
+			(at 44.45 38.1 0)
+			(effects
+				(font
+					(size 1.27 1.27)
+				)
+			)
+		)
+		(property "Footprint" ""
+			(at 44.45 43.18 0)
+			(effects
+				(font
+					(size 1.27 1.27)
+				)
+				(hide yes)
+			)
+		)
+		(property "Datasheet" "~"
+			(at 44.45 43.18 0)
+			(effects
+				(font
+					(size 1.27 1.27)
+				)
+				(hide yes)
+			)
+		)
+		(property "Description" "Special symbol for telling ERC where power comes from"
+			(at 44.45 43.18 0)
+			(effects
+				(font
+					(size 1.27 1.27)
+				)
+				(hide yes)
+			)
+		)
+		(pin "1"
+		)
+		(instances
+			(project ""
+				(path "/79a95597-2db4-4373-9cc6-70296586f172"
+					(reference "#FLG03")
+					(unit 1)
+				)
