File: OscilloscopeV1/_autosave-Projet_s6_oscillovpresquefinal.kicad_pcb (KiCad board)
At the start: 2 copper layers, 43.5 x 74.6 mm, 33 parts, among them IC1 PGA849RGTR, J1 Conn_Coaxial, J2 Conn_01x06_Socket, J3 PILES_3AA, J4 Conn_01x05_Pin, SW1 SW_SPST, U1 MCP1826S, U3 AP2112K-3.3, U4 STM32L476RGTx

Commit message: Point de départ du routage
Parts:
- C13, C14, C4, C5: moved to F.Cu
- moved U1 5.02 mm to (150.2, 90.2)
- moved C5 4.70 mm to (151.0, 100.5)
- moved C13 3.40 mm to (151.0, 108.2)
