File: OscilloscopeV1/Projet_s6_oscillovpresquefinal.kicad_pcb (KiCad board)
At the start: 2 copper layers, 43.5 x 74.6 mm, 33 parts, among them IC1 PGA849RGTR, J1 Conn_Coaxial, J2 Conn_01x06_Socket, J3 PILES_3AA, J4 Conn_01x05_Pin, SW1 SW_SPST, U1 MCP1826S, U3 AP2112K-3.3, U4 STM32L476RGTx

Commit message: PCB Final
Parts:
- removed C4: 10µ, Capacitor_SMD:CP_Elec_4x5.7
- removed H3, H4: MountingHole_Pad, MountingHole:MountingHole_3.2mm_M3_DIN965_Pad
- C1, C10, C11, C12, C13, C14, C2, C3, C5, C6, C7, C8, C9, D1, D2, D3, R1, R2: moved to F.Cu
- moved H1 86.3 mm to (229.4, 38.4)
- moved H2 82.2 mm to (213.3, 126.3)
- moved U1 81.0 mm to (228.1, 71.1), turned to 90 degrees
- moved C6 77.5 mm to (228.5, 91.5), turned to -90 degrees
- moved C13 77.1 mm to (223.4, 78.4), turned to 180 degrees
- moved C10 76.1 mm to (228.5, 96.7)
- moved PS1 76.0 mm to (224.3, 56.5)
- moved C7 73.7 mm to (225.3, 84.0)
- moved J1 73.4 mm to (220.4, 40.8)
- moved R1 72.9 mm to (218.8, 72.9)
- moved C8 71.9 mm to (230.1, 88.5), turned to 0 degrees
- moved D1 71.2 mm to (222.4, 73.9), turned to -90 degrees
- moved J2 68.8 mm to (218.3, 119.1)
- moved C5 64.9 mm to (213.5, 78.3)
- moved C11 62.7 mm to (214.7, 85.5), turned to 0 degrees
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Routing:
- net GND: track 0.00 -> 193.1 mm, vias 0 -> 5
- net V3.3_DIG: track 0.00 -> 119.0 mm, vias 0 -> 1
- net Sortie5V: track 0.00 -> 64.1 mm
- net Net-(IC1-IN-): track 0.00 -> 44.8 mm
- net BAT_PLUS: track 0.00 -> 41.1 mm, vias 0 -> 1
- net KEY: track 0.00 -> 37.4 mm, vias 0 -> 1
- net Net-(IC1-IN+): track 0.00 -> 28.8 mm
- net UART_TX: track 0.00 -> 24.4 mm, vias 0 -> 2
- net UART_RX: track 0.00 -> 24.0 mm, vias 0 -> 2
- net Entree_adc: track 0.00 -> 23.2 mm, vias 0 -> 2
- net Vref_1.5: track 0.00 -> 22.1 mm
- net ANL0: track 0.00 -> 21.9 mm, vias 0 -> 3
- net ANL1: track 0.00 -> 21.9 mm, vias 0 -> 2
- net ANL2: track 0.00 -> 21.0 mm, vias 0 -> 2
- net Traco_-15V: track 0.00 -> 20.2 mm
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- added copper zone on B.Cu, net (none)
- added copper zone on F.Cu, net (none)
- removed copper zone on B.Cu, net GND
- removed copper zone on F.Cu, net GND
Other:
- board size 43.5 x 74.6 mm -> 22.9 x 94.7 mm
