File: OscilloscopeV1/Projet_s6_oscillovpresquefinal.kicad_pcb (KiCad board)
At the start: 2 copper layers, 23.6 x 94.7 mm, 30 parts, among them IC1 PGA849RGTR, J1 Conn_Coaxial, J2 Conn_01x06_Socket, J3 PILES_3AA, J4 Conn_01x05_Pin, SW1 SW_SPST, U1 MCP1826S, U3 AP2112K-3.3, U4 STM32L476RGTx

Commit message: Add fabrication files
Other:
- board text added: "G. Boudoux D. Oscillo wireless"
Changed lines of the file:
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@@
 		(layer "Edge.Cuts")
+	)
+	(gr_text "G. Boudoux D.\nOscillo wireless"
+		(at 214 51 90)
+		(layer "F.SilkS")
+		(effects
+			(font
+				(size 1 1)
+				(thickness 0.15)
+			)
+			(justify left bottom)
+		)
 	)
 	(segment
