File: OscilloscopeV1/Projet_s6_oscillovpresquefinal-backups/Projet_s6_oscillovpresquefinal.kicad_pcb (KiCad board)
At the start: 2 copper layers, 23.6 x 94.7 mm, 30 parts, among them IC1 PGA849RGTR, J1 Conn_Coaxial, J2 Conn_01x06_Socket, J3 PILES_3AA, J4 Conn_01x05_Pin, SW1 SW_SPST, U1 MCP1826S, U3 AP2112K-3.3, U4 STM32L476RGTx

Commit message: Add files via upload
Parts:
- moved C2 1.10 mm to (221.9, 68.7), turned to 180 degrees
- moved H2 0.94 mm to (213.4, 126.2)
- moved J2 0.68 mm to (218.3, 119.1)
- moved H1 0.60 mm to (229.3, 38.6)
- moved J1 0.55 mm to (220.4, 40.8)
Routing:
- net GND: track 66.1 -> 220.2 mm, vias 0 -> 5
- net V3.3_DIG: track 116.1 -> 113.8 mm, vias 6 -> 4
- net Traco_-15V: track 18.7 -> 20.2 mm
- net ANL2: track 25.6 -> 24.7 mm
- net Net-(IC1-EP): track 5.84 -> 5.11 mm
- net KEY: track 38.1 -> 37.4 mm
- net UART_TX: track 24.8 -> 24.4 mm, vias 0 -> 2
- net UART_RX: track 23.8 -> 24.0 mm, vias 0 -> 2
- added copper zone on B.Cu, net (none)
- added copper zone on F.Cu, net (none)
- removed copper zone on B.Cu, net GND
- removed copper zone on F.Cu, net GND
Other:
- board size 23.6 x 94.7 mm -> 22.9 x 94.7 mm
