File: OscilloscopeV1/Projet_s6_oscillovpresquefinal-backups/Projet_s6_oscillovpresquefinal.kicad_sch (KiCad schematic)
At the start: 31 parts, among them IC1 PGA849RGTR, J1 Conn_Coaxial, J2 Conn_01x06_Socket, J3 PILES_3AA, J4 Conn_01x05_Pin, SW1 SW_SPST, U1 MCP1826S, U3 AP2112K-3.3, U4 STM32L476RGTx

Commit message: Add files via upload
Parts:
- added H3, H4: MountingHole_Pad, MountingHole:MountingHole_3.2mm_M3_DIN965_Pad, symbol Mechanical:MountingHole_Pad
Connections:
- net GND: now also H3.1, H4.1
Changed lines of the file:
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@@
 	)
 	(junction
+		(at 292.1 224.79)
+		(diameter 0)
+		(color 0 0 0 0)
+	)
+	(junction
 		(at 364.49 72.39)
 		(diameter 0)
@@
 	)
 	(junction
+		(at 292.1 229.87)
+		(diameter 0)
+		(color 0 0 0 0)
+	)
+	(junction
 		(at 326.39 81.28)
 		(diameter 0)
@@
 	(wire
 		(pts
+			(xy 292.1 224.79) (xy 292.1 219.71)
+		)
+		(stroke
+			(width 0)
+			(type default)
+		)
+	)
+	(wire
+		(pts
 			(xy 365.76 224.79) (xy 374.65 224.79)
 		)
@@
 	(wire
 		(pts
+			(xy 292.1 229.87) (xy 292.1 233.68)
+		)
+		(stroke
+			(width 0)
+			(type default)
+		)
+	)
+	(wire
+		(pts
 			(xy 170.18 205.74) (xy 170.18 207.01)
 		)
@@
 	(wire
 		(pts
+			(xy 292.1 224.79) (xy 297.18 224.79)
+		)
+		(stroke
+			(width 0)
+			(type default)
+		)
+	)
+	(wire
+		(pts
 			(xy 128.27 58.42) (xy 128.27 64.77)
 		)
@@
 	(wire
 		(pts
-			(xy 292.1 219.71) (xy 292.1 233.68)
+			(xy 297.18 229.87) (xy 292.1 229.87)
+		)
+		(stroke
+			(width 0)
+			(type default)
+		)
+	)
+	(wire
+		(pts
+			(xy 292.1 224.79) (xy 292.1 229.87)
 		)
 		(stroke
@@
 	)
 	(symbol
+		(lib_id "Mechanical:MountingHole_Pad")
+		(at 299.72 229.87 270)
+		(unit 1)
+		(exclude_from_sim no)
+		(in_bom no)
+		(on_board yes)
+		(dnp no)
+		(fields_autoplaced yes)
+		(property "Reference" "H4"
+			(at 303.53 228.5999 90)
+			(effects
+				(font
+					(size 1.27 1.27)
+				)
+				(justify left)
+			)
+		)
+		(property "Value" "MountingHole_Pad"
+			(at 303.53 231.1399 90)
+			(effects
+				(font
+					(size 1.27 1.27)
+				)
+				(justify left)
+			)
+		)
+		(property "Footprint" "MountingHole:MountingHole_3.2mm_M3_DIN965_Pad"
+			(at 299.72 229.87 0)
+			(effects
+				(font
+					(size 1.27 1.27)
+				)
+				(hide yes)
+			)
+		)
+		(property "Datasheet" "~"
+			(at 299.72 229.87 0)
+			(effects
+				(font
+					(size 1.27 1.27)
+				)
+				(hide yes)
+			)
+		)
+		(property "Description" "Mounting Hole with connection"
+			(at 299.72 229.87 0)
+			(effects
+				(font
+					(size 1.27 1.27)
+				)
+				(hide yes)
+			)
+		)
+		(pin "1"
+		)
+		(instances
+			(project "Projet_s6_oscillovpresquefinal"
+				(path "/79a95597-2db4-4373-9cc6-70296586f172"
+					(reference "H4")
+					(unit 1)
+				)
+			)
+		)
+	)
+	(symbol
 		(lib_id "Device:C_Small")
 		(at 353.06 66.04 0)
@@
 					(unit 1)
 				)
+			)
+		)
+	)
+	(symbol
+		(lib_id "Mechanical:MountingHole_Pad")
+		(at 299.72 224.79 270)
+		(unit 1)
+		(exclude_from_sim no)
+		(in_bom no)
+		(on_board yes)
+		(dnp no)
+		(fields_autoplaced yes)
+		(property "Reference" "H3"
+			(at 303.53 223.5199 90)
+			(effects
+				(font
+					(size 1.27 1.27)
+				)
+				(justify left)
+			)
+		)
+		(property "Value" "MountingHole_Pad"
+			(at 303.53 226.0599 90)
+			(effects
+				(font
+					(size 1.27 1.27)
+				)
+				(justify left)
+			)
+		)
+		(property "Footprint" "MountingHole:MountingHole_3.2mm_M3_DIN965_Pad"
+			(at 299.72 224.79 0)
+			(effects
+				(font
+					(size 1.27 1.27)
+				)
+				(hide yes)
+			)
+		)
+		(property "Datasheet" "~"
+			(at 299.72 224.79 0)
+			(effects
+				(font
+					(size 1.27 1.27)
+				)
+				(hide yes)
+			)
+		)
+		(property "Description" "Mounting Hole with connection"
+			(at 299.72 224.79 0)
+			(effects
+				(font
+					(size 1.27 1.27)
+				)
+				(hide yes)
+			)
+		)
+		(pin "1"
+		)
+		(instances
+			(project "Projet_s6_oscillovpresquefinal"
+				(path "/79a95597-2db4-4373-9cc6-70296586f172"
+					(reference "H3")
+					(unit 1)
+				)
